File: ealge_files/TopBoardLidar.sch (EAGLE design)
At the start: 15 parts, among them U2 52207-0485, U3 VL53L1XSMD

Commit message: completed top board; started bottom borad
Other:
- note added: "open hardware"
- note removed: "/home/pratique/Downloads/prg-white (1).bmp"
Changed lines of the file:
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@@
 <rectangle x1="-38.8239" y1="-30.5943" x2="-38.7477" y2="-30.5181" layer="94"/>
 <rectangle x1="-38.6715" y1="-30.5943" x2="-38.1381" y2="-30.5181" layer="94"/>
-<text x="-64.3128" y="-56.007" size="0.1524" layer="200" font="vector">/home/pratique/Downloads/prg-white (1).bmp</text>
+<text x="-60.96" y="-55.88" size="2.54" layer="94" ratio="5" distance="59">open hardware</text>
 </plain>
 <instances>

Commit message: completed bottom layer.. and started with nanopi shield
Connections:
- net GND: now also U2.5, U2.6
Changed lines of the file:
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@@
 <part name="LOGO1" library="SparkFun-Aesthetics" deviceset="OSHW-LOGO" device="MINI"/>
 <part name="U$1" library="SparkX" deviceset="SPARKX-LOGO" device="4"/>
+<part name="GND2" library="SparkFun-PowerSymbols" library_urn="urn:adsk.eagle:library:530" deviceset="GND" device=""/>
+<part name="GND3" library="SparkFun-PowerSymbols" library_urn="urn:adsk.eagle:library:530" deviceset="GND" device=""/>
 </parts>
 <sheets>
@@
 <instance part="LOGO1" gate="G$1" x="-88.9" y="-35.56" smashed="yes"/>
 <instance part="U$1" gate="G$1" x="-88.9" y="-50.8" smashed="yes"/>
+<instance part="GND2" gate="1" x="-17.78" y="0" smashed="yes">
+<attribute name="VALUE" x="-17.78" y="-0.254" size="1.778" layer="96" align="top-center"/>
+</instance>
+<instance part="GND3" gate="1" x="-81.28" y="0" smashed="yes">
+<attribute name="VALUE" x="-81.28" y="-0.254" size="1.778" layer="96" align="top-center"/>
+</instance>
 </instances>
 <busses>
@@
 <wire x1="-25.4" y1="-7.62" x2="-25.4" y2="-10.16" width="0.1524" layer="91"/>
 </segment>
+<segment>
+<pinref part="U2" gate="A" pin="6"/>
+<wire x1="-68.58" y1="-2.54" x2="-68.58" y2="7.62" width="0.1524" layer="91"/>
+<wire x1="-68.58" y1="7.62" x2="-81.28" y2="7.62" width="0.1524" layer="91"/>
+<pinref part="GND3" gate="1" pin="GND"/>
+<wire x1="-81.28" y1="7.62" x2="-81.28" y2="2.54" width="0.1524" layer="91"/>
+</segment>
+<segment>
+<pinref part="GND2" gate="1" pin="GND"/>
+<wire x1="-17.78" y1="2.54" x2="-30.48" y2="2.54" width="0.1524" layer="91"/>
+<wire x1="-30.48" y1="2.54" x2="-30.48" y2="-2.54" width="0.1524" layer="91"/>
+<pinref part="U2" gate="A" pin="5"/>
+<wire x1="-30.48" y1="-2.54" x2="-33.02" y2="-2.54" width="0.1524" layer="91"/>
+</segment>
 </net>
